Commit message: re-added cameras on multi-drones

File: sjtu_drone_description/urdf/sjtu_drone_multi.urdf.xacro (robot description, xacro)
@@ -24,8 +24,21 @@
     </visual>
   </link>
+  <joint name="${drone_id}/front_cam_joint" type="fixed">
+    <origin rpy="0 0 0" xyz="0.2 0 0"/>
+    <parent link="${drone_id}/base_link" />
+    <child link="${drone_id}/front_cam_link" />
+  </joint>
+  <link name="${drone_id}/front_cam_link"/>
+  <joint name="${drone_id}/bottom_cam_joint" type="fixed">
+    <origin rpy="0 1.570796326794897 0" xyz="0 0 0"/>
+    <parent link="${drone_id}/base_link" />
+    <child link="${drone_id}/bottom_cam_link" />
+  </joint>
+  <link name="${drone_id}/bottom_cam_link"/>
   <gazebo>
     <plugin name='simple_drone' filename='libplugin_drone.so'>
-      <bodyName>base_link</bodyName>
-      <rosNamespace>drone</rosNamespace>
+      <bodyName>${drone_id}/base_link</bodyName>
+      <rosNamespace>${drone_id}</rosNamespace>
+      <imuTopic>${drone_id}/imu</imuTopic>
       <rollpitchProportionalGain>10.0</rollpitchProportionalGain>
       <rollpitchDifferentialGain>5.0</rollpitchDifferentialGain>
@@ -55,3 +68,96 @@
     </plugin>
   </gazebo>
+  <!-- Sensors -->
+  <!-- IMU sensor in 100fps -->
+  <gazebo reference="${drone_id}/base_link">
+    <sensor name='sensor_imu' type='imu'>
+      <always_on> 1 </always_on>
+      <visualize>1</visualize>
+      <update_rate> 100 </update_rate>
+      <pose> 0 0 0 0 0 0 </pose>
+      <plugin name='imu' filename='libgazebo_ros_imu_sensor.so'>
+        <initial_orientation_as_reference>false</initial_orientation_as_reference>
+      </plugin>
+      <imu>
+        <noise>
+          <type>gaussian</type>
+          <rate>
+            <mean> 0 </mean>
+            <stddev> 0 </stddev>
+          </rate>
+          <accel>
+            <mean> 0 </mean>
+            <stddev> 0.00 </stddev>
+          </accel>
+        </noise>
+      </imu>
+    </sensor>
+  </gazebo>
+ <gazebo reference="${drone_id}/front_cam_link">
+    <sensor name="front_camera" type="camera">
+      <camera>
+        <horizontal_fov>2.09</horizontal_fov>
+        <image>
+          <width>640</width>
+          <height>360</height>
+          <format>R8G8B8</format>
+        </image>
+        <clip>
+          <near>0.1</near>
+          <far>100</far>
+        </clip>
+        <noise>
+          <type>gaussian</type>
+          <mean>0.0</mean>
+          <stddev>0.005</stddev>
+        </noise>
+      </camera>
+      <always_on>1</always_on>
+      <update_rate>60</update_rate>
+      <visualize>true</visualize>
+      <plugin name="camera_front" filename="libgazebo_ros_camera.so">
+        <ros>
+          <remapping>image_raw:=camera_front</remapping>
+          <remapping>camera_info:=camera_front_info</remapping>
+        </ros>
+        <camera_name>front</camera_name>
+        <frame_name>front_cam_link</frame_name>
+        <hack_baseline>0.07</hack_baseline>
+      </plugin>
+    </sensor>
+  </gazebo>
+  <!-- downward looking camera -->
+  <gazebo reference="${drone_id}/bottom_cam_link">
+    <sensor name="down_camera" type="camera">
+      <camera>
+        <horizontal_fov>1.047</horizontal_fov>
+        <image>
+          <width>640</width>
+          <height>360</height>
+          <format>R8G8B8</format>
+        </image>
+        <clip>
+          <near>0.1</near>
+          <far>100</far>
+        </clip>
+        <noise>
+          <type>gaussian</type>
+          <mean>0.0</mean>
+          <stddev>0.005</stddev>
+        </noise>
+      </camera>
+      <always_on>1</always_on>
+      <update_rate>15</update_rate>
+      <visualize>true</visualize>
+      <plugin name="camera_bottom" filename="libgazebo_ros_camera.so">
+        <ros>
+          <remapping>image_raw:=camera_bottom</remapping>
+          <remapping>camera_info:=camera_bottom_info</remapping>
+        </ros>
+        <camera_name>bottom</camera_name>
+        <frame_name>bottom_cam_link</frame_name>
+        <hack_baseline>0.07</hack_baseline>
+      </plugin>
+    </sensor>
+  </gazebo>
 </robot>

Commit message: change to 15 degree downwards tilt on forwards camera

File: sjtu_drone_description/urdf/sjtu_drone_multi.urdf.xacro (robot description, xacro)
@@ -25,5 +25,5 @@
   </link>
   <joint name="${drone_id}/front_cam_joint" type="fixed">
-    <origin rpy="0 0 0" xyz="0.2 0 0"/>
+    <origin rpy="0 0.261799 0" xyz="0.2 0 0"/>
     <parent link="${drone_id}/base_link" />
     <child link="${drone_id}/front_cam_link" />

Commit message: feat: changed camera params for stereoscopic vision

File: sjtu_drone_description/urdf/sjtu_drone_multi.urdf.xacro (robot description, xacro)
@@ -24,16 +24,16 @@
     </visual>
   </link>
-  <joint name="${drone_id}/front_cam_joint" type="fixed">
-    <origin rpy="0 0.261799 0" xyz="0.2 0 0"/>
+  <joint name="${drone_id}/left_cam_joint" type="fixed">
+    <origin rpy="0 0.25 0" xyz="0.2 0.05 0"/>
     <parent link="${drone_id}/base_link" />
-    <child link="${drone_id}/front_cam_link" />
+    <child link="${drone_id}/left_cam_link" />
   </joint>
-  <link name="${drone_id}/front_cam_link"/>
-  <joint name="${drone_id}/bottom_cam_joint" type="fixed">
-    <origin rpy="0 1.570796326794897 0" xyz="0 0 0"/>
+  <link name="${drone_id}/left_cam_link"/>
+  <joint name="${drone_id}/right_cam_joint" type="fixed">
+    <origin rpy="0 0.25 0" xyz="0.2 -0.05 0"/>
     <parent link="${drone_id}/base_link" />
-    <child link="${drone_id}/bottom_cam_link" />
+    <child link="${drone_id}/right_cam_link" />
   </joint>
-  <link name="${drone_id}/bottom_cam_link"/>
+  <link name="${drone_id}/right_cam_link"/>
   <gazebo>
     <plugin name='simple_drone' filename='libplugin_drone.so'>
@@ -94,8 +94,9 @@
     </sensor>
   </gazebo>
- <gazebo reference="${drone_id}/front_cam_link">
-    <sensor name="front_camera" type="camera">
+  <!-- left camera -->
+ <gazebo reference="${drone_id}/left_cam_link">
+    <sensor name="left_camera" type="camera">
       <camera>
-        <horizontal_fov>2.09</horizontal_fov>
+        <horizontal_fov>1.2</horizontal_fov>
         <image>
           <width>960</width>
@@ -110,5 +111,5 @@
           <type>gaussian</type>
           <mean>0.0</mean>
-          <stddev>0.005</stddev>
+          <stddev>0.001</stddev>
         </noise>
       </camera>
@@ -116,23 +117,23 @@
       <update_rate>60</update_rate>
       <visualize>true</visualize>
-      <plugin name="camera_front" filename="libgazebo_ros_camera.so">
+      <plugin name="camera_left" filename="libgazebo_ros_camera.so">
         <ros>
-          <remapping>image_raw:=camera_front</remapping>
-          <remapping>camera_info:=camera_front_info</remapping>
+          <remapping>image_raw:=camera_left</remapping>
+          <remapping>camera_info:=camera_left_info</remapping>
         </ros>
-        <camera_name>front</camera_name>
-        <frame_name>front_cam_link</frame_name>
-        <hack_baseline>0.07</hack_baseline>
+        <camera_name>left</camera_name>
+        <frame_name>left_cam_link</frame_name>
+        <hack_baseline>0.1</hack_baseline>
       </plugin>
     </sensor>
   </gazebo>
-  <!-- downward looking camera -->
-  <gazebo reference="${drone_id}/bottom_cam_link">
-    <sensor name="down_camera" type="camera">
+  <!-- right camera -->
+  <gazebo reference="${drone_id}/right_cam_link">
+    <sensor name="right_camera" type="camera">
       <camera>
-        <horizontal_fov>1.047</horizontal_fov>
+        <horizontal_fov>1.2</horizontal_fov>
         <image>
-          <width>640</width>
-          <height>360</height>
+          <width>960</width>
+          <height>540</height>
           <format>R8G8B8</format>
         </image>
@@ -144,18 +145,18 @@
           <type>gaussian</type>
           <mean>0.0</mean>
-          <stddev>0.005</stddev>
+          <stddev>0.001</stddev>
         </noise>
       </camera>
       <always_on>1</always_on>
-      <update_rate>15</update_rate>
+      <update_rate>60</update_rate>
       <visualize>true</visualize>
-      <plugin name="camera_bottom" filename="libgazebo_ros_camera.so">
+      <plugin name="camera_right" filename="libgazebo_ros_camera.so">
         <ros>
-          <remapping>image_raw:=camera_bottom</remapping>
-          <remapping>camera_info:=camera_bottom_info</remapping>
+          <remapping>image_raw:=camera_right</remapping>
+          <remapping>camera_info:=camera_right_info</remapping>
         </ros>
-        <camera_name>bottom</camera_name>
-        <frame_name>bottom_cam_link</frame_name>
-        <hack_baseline>0.07</hack_baseline>
+        <camera_name>right</camera_name>
+        <frame_name>right_cam_link</frame_name>
+        <hack_baseline>0.1</hack_baseline>
       </plugin>
     </sensor>
